Commit message: Correct script, Fix root joint as anchor movable in URDF

File: urdf/baxter_original.urdf (robot description, URDF)
Before this commit: robot baxter, 48 links, 47 joints
Links:
- removed link base_link
- added link dummyhead1, mass 0.0001
- added link head_camera, mass 0.0001
Joints:
- removed joint j_base_link
- added joint dummy: type fixed, parent head, child dummyhead1, origin xyz=0 0 0 rpy=0 0 0
- added joint head_camera: type fixed, parent head, child head_camera, origin xyz=0.12839 0 0.06368 rpy=1.75057 0 1.57079632679
- joint pedestal_fixed: parent base -> torso
- joint torso_t0: axis 0 0 1 -> (none); limit lower=-1.8 upper=1.8 effort=50000 velocity=10000 -> lower=-3.01 upper=3.01 effort=50000 velocity=10000; type revolute -> fixed
