Commit message: Fix baxter URDF, update script to TADR2, add convergence graphs

File: urdf/baxter.urdf (robot description, URDF)
Before this commit: robot baxter, 48 links, 47 joints
Links:
- link head: geometry collision mesh filename=package://baxter_description/meshes/head/H0.DAE; visual mesh filename=package://baxter_description/meshes/head/H0.DAE
- link left_lower_elbow: geometry collision mesh filename=package://baxter_description/meshes/lower_elbow/E1.DAE; visual mesh filename=package://baxter_description/meshes/lower_elbow/E1.DAE
- link left_lower_forearm: geometry collision mesh filename=package://baxter_description/meshes/lower_forearm/W1.DAE; visual mesh filename=package://baxter_description/meshes/lower_forearm/W1.DAE
- link left_lower_shoulder: geometry collision mesh filename=package://baxter_description/meshes/lower_shoulder/S1.DAE; visual mesh filename=package://baxter_description/meshes/lower_shoulder/S1.DAE
- link left_upper_elbow: geometry collision mesh filename=package://baxter_description/meshes/upper_elbow/E0.DAE; visual mesh filename=package://baxter_description/meshes/upper_elbow/E0.DAE
- link left_upper_forearm: geometry collision mesh filename=package://baxter_description/meshes/upper_forearm/W0.DAE; visual mesh filename=package://baxter_description/meshes/upper_forearm/W0.DAE
- link left_upper_shoulder: geometry collision mesh filename=package://baxter_description/meshes/upper_shoulder/S0.DAE; visual mesh filename=package://baxter_description/meshes/upper_shoulder/S0.DAE
- link left_wrist: geometry collision mesh filename=package://baxter_description/meshes/wrist/W2.DAE; visual mesh filename=package://baxter_description/meshes/wrist/W2.DAE
- link right_lower_elbow: geometry collision mesh filename=package://baxter_description/meshes/lower_elbow/E1.DAE; visual mesh filename=package://baxter_description/meshes/lower_elbow/E1.DAE
- link right_lower_forearm: geometry collision mesh filename=package://baxter_description/meshes/lower_forearm/W1.DAE; visual mesh filename=package://baxter_description/meshes/lower_forearm/W1.DAE
- link right_lower_shoulder: geometry collision mesh filename=package://baxter_description/meshes/lower_shoulder/S1.DAE; visual mesh filename=package://baxter_description/meshes/lower_shoulder/S1.DAE
- link right_upper_elbow: geometry collision mesh filename=package://baxter_description/meshes/upper_elbow/E0.DAE; visual mesh filename=package://baxter_description/meshes/upper_elbow/E0.DAE
- link right_upper_forearm: geometry collision mesh filename=package://baxter_description/meshes/upper_forearm/W0.DAE; visual mesh filename=package://baxter_description/meshes/upper_forearm/W0.DAE
- link right_upper_shoulder: geometry collision mesh filename=package://baxter_description/meshes/upper_shoulder/S0.DAE; visual mesh filename=package://baxter_description/meshes/upper_shoulder/S0.DAE
- link right_wrist: geometry collision mesh filename=package://baxter_description/meshes/wrist/W2.DAE; visual mesh filename=package://baxter_description/meshes/wrist/W2.DAE
- link screen: geometry collision mesh filename=package://baxter_description/meshes/head/H1.DAE; visual mesh filename=package://baxter_description/meshes/head/H1.DAE
- link sonar_ring: geometry collision cylinder length=0.01 radius=0.085; visual cylinder length=0.01 radius=0.085
